Commit message: Add a nicer URDF model and visualize it

File: urdf/cabot.urdf (robot description, URDF)
Before this commit: robot cabot, 3 links, 2 joints
Links:
- added link kinect_link; visual box size=0.07 0.25 0.06
- link base_link: geometry visual box size=0.49 0.30 0.43
- link imu_link: geometry 
Joints:
- removed joint laser_link_joint
- added joint kinect_link_joint: type fixed, parent base_link, child kinect_link, origin xyz=0.165 0 0.46
- added joint laser_kinect_joint: type fixed, parent kinect_link, child laser_link, origin xyz=0 0.08 0.09

Commit message: Updated URDF for new lidar location

File: urdf/cabot.urdf (robot description, URDF)
Before this commit: robot cabot, 4 links, 3 joints
Links:
- link base_link: geometry visual box size=0.55 0.30 0.46
Joints:
- joint kinect_link_joint: origin xyz=0.165 0 0.46 -> xyz=0.225 0 0.46
- joint laser_kinect_joint: origin xyz=0 0.08 0.09 -> xyz=0.08 -0.06 -0.15
